File: FuzzWah.kicad_pcb (KiCad board)
At the start: 2 copper layers, 0 parts

Commit message: Adctualización de PCB
Parts:
- added C1: 10uF, Capacitor_THT:CP_Radial_D5.0mm_P2.00mm, F.Cu at (202.1, 37.5)
- added C10: 10uF, Capacitor_THT:CP_Radial_D5.0mm_P2.00mm, F.Cu at (147.4, 57.1)
- added C11: 10uF, Capacitor_THT:CP_Radial_D5.0mm_P2.00mm, F.Cu at (210.8, 84.0)
- added C12: 1nF, Capacitor_THT:C_Disc_D5.1mm_W3.2mm_P5.00mm, F.Cu at (210.1, 102.8)
- added C13: 100nF, Capacitor_THT:C_Disc_D5.1mm_W3.2mm_P5.00mm, F.Cu at (210.1, 107.5)
- added C14: 10uF, Capacitor_THT:CP_Radial_D5.0mm_P2.00mm, F.Cu at (210.8, 90.5)
- added C15: 10uF, Capacitor_THT:CP_Radial_D5.0mm_P2.00mm, F.Cu at (210.8, 97.1)
- added C16: 10nF, Capacitor_THT:C_Disc_D5.1mm_W3.2mm_P5.00mm, F.Cu at (170.2, 36.5)
- added C17: 10uF, Capacitor_THT:CP_Radial_D5.0mm_P2.00mm, F.Cu at (179.1, 49.0)
- added C18: 30nF, Capacitor_THT:C_Disc_D5.1mm_W3.2mm_P5.00mm, F.Cu at (170.2, 41.3)
- added C19: 200nF, Capacitor_THT:C_Disc_D5.1mm_W3.2mm_P5.00mm, F.Cu at (170.2, 46.0)
- added C2: 2nF, Capacitor_THT:C_Disc_D5.1mm_W3.2mm_P5.00mm, F.Cu at (201.3, 56.2)
- added C20: 200nF, Capacitor_THT:C_Disc_D5.1mm_W3.2mm_P5.00mm, F.Cu at (170.2, 50.8)
- added C21: 10uF, Capacitor_THT:CP_Radial_D5.0mm_P2.00mm, F.Cu at (147.4, 63.6)
- added C22: 10uF, Capacitor_THT:CP_Radial_D5.0mm_P2.00mm, F.Cu at (188.8, 113.3)
- added C3: 10uF, Capacitor_THT:CP_Radial_D5.0mm_P2.00mm, F.Cu at (202.1, 44.0)
- added C4: 10uF, Capacitor_THT:CP_Radial_D5.0mm_P2.00mm, F.Cu at (202.1, 50.5)
- added C5: 100nF, Capacitor_THT:C_Disc_D5.1mm_W3.2mm_P5.00mm, F.Cu at (201.3, 61.0)
- added C6: 10uF, Capacitor_THT:CP_Radial_D5.0mm_P2.00mm, F.Cu at (147.4, 37.5)
- added C7: 10uF, Capacitor_THT:CP_Radial_D5.0mm_P2.00mm, F.Cu at (147.4, 44.0)
- added C8: 100nF, Capacitor_THT:C_Disc_D5.1mm_W3.2mm_P5.00mm, F.Cu at (188.0, 100.5)
- added C9: 10uF, Capacitor_THT:CP_Radial_D5.0mm_P2.00mm, F.Cu at (147.4, 50.5)
- added D1: 1N4148, Diode_THT:D_DO-35_SOD27_P7.62mm_Horizontal, F.Cu at (146.6, 86.1)
- added D2: 1N4148, Diode_THT:D_DO-35_SOD27_P7.62mm_Horizontal, F.Cu at (146.6, 89.6)
- added J1: BYPASS, Connector_PinHeader_2.54mm:PinHeader_1x06_P2.54mm_Vertical, F.Cu at (229.5, 95.3)
- added J2: WAH, Connector_PinHeader_2.54mm:PinHeader_1x06_P2.54mm_Vertical, F.Cu at (256.2, 95.6)
- added J3: INPUT, Connector_Audio:Jack_6.35mm_Neutrik_NMJ6HCD3_Horizontal, F.Cu at (73.2, 58.3)
- added J4: OUTPUT, Connector_Audio:Jack_6.35mm_Neutrik_NMJ6HCD3_Horizontal, F.Cu at (16.8, 58.3)
- added J5: PWR, Connector_PinHeader_2.54mm:PinHeader_1x02_P2.54mm_Vertical, F.Cu at (50.8, 45.7)
- added L1: 500uH, Inductor_THT:L_Radial_D16.8mm_P11.43mm_Vishay_IHB-1, F.Cu at (172.1, 62.4)
- added Q1: 2N3904, Package_TO_SOT_THT:TO-92_Inline, F.Cu at (208.3, 37.4)
- added Q2: 2N3904, Package_TO_SOT_THT:TO-92_Inline, F.Cu at (208.3, 43.2)
- added Q3: 2N3904, Package_TO_SOT_THT:TO-92_Inline, F.Cu at (147.1, 70.2)
- added Q4: 2N3904, Package_TO_SOT_THT:TO-92_Inline, F.Cu at (147.1, 76.0)
- added Q5: 2N3904, Package_TO_SOT_THT:TO-92_Inline, F.Cu at (147.1, 81.8)
- added Q6: 2N3904, Package_TO_SOT_THT:TO-92_Inline, F.Cu at (210.5, 113.1)
- added Q7: 2N3904, Package_TO_SOT_THT:TO-92_Inline, F.Cu at (178.7, 37.4)
- added Q8: 2N3904, Package_TO_SOT_THT:TO-92_Inline, F.Cu at (178.7, 43.2)
- added R1: 47K, Resistor_THT:R_Axial_DIN0207_L6.3mm_D2.5mm_P7.62mm_Horizontal, F.Cu at (190.5, 36.2)
- added R10: 10K, Resistor_THT:R_Axial_DIN0207_L6.3mm_D2.5mm_P7.62mm_Horizontal, F.Cu at (135.9, 36.2)
- added R101: 1M, Resistor_THT:R_Axial_DIN0207_L6.3mm_D2.5mm_P7.62mm_Horizontal, F.Cu at (190.5, 72.7)
- added R102: 1M, Resistor_THT:R_Axial_DIN0207_L6.3mm_D2.5mm_P7.62mm_Horizontal, F.Cu at (135.9, 84.8)
- added R103: 100K, Resistor_THT:R_Axial_DIN0207_L6.3mm_D2.5mm_P7.62mm_Horizontal, F.Cu at (135.9, 88.8)
- added R104: 1M, Resistor_THT:R_Axial_DIN0207_L6.3mm_D2.5mm_P7.62mm_Horizontal, F.Cu at (199.3, 119.2)
- added R105: 0R, Resistor_THT:R_Axial_DIN0207_L6.3mm_D2.5mm_P7.62mm_Horizontal, F.Cu at (135.9, 92.9)
- added R11: 220K, Resistor_THT:R_Axial_DIN0207_L6.3mm_D2.5mm_P7.62mm_Horizontal, F.Cu at (135.9, 40.2)
- added R12: 10K, Resistor_THT:R_Axial_DIN0207_L6.3mm_D2.5mm_P7.62mm_Horizontal, F.Cu at (135.9, 44.3)
- added R13: 100K, Resistor_THT:R_Axial_DIN0207_L6.3mm_D2.5mm_P7.62mm_Horizontal, F.Cu at (135.9, 48.4)
- added R14: 470R, Resistor_THT:R_Axial_DIN0207_L6.3mm_D2.5mm_P7.62mm_Horizontal, F.Cu at (135.9, 52.4)
- added R15: 22K, Resistor_THT:R_Axial_DIN0207_L6.3mm_D2.5mm_P7.62mm_Horizontal, F.Cu at (135.9, 56.5)
- added R16: 1K8, Resistor_THT:R_Axial_DIN0207_L6.3mm_D2.5mm_P7.62mm_Horizontal, F.Cu at (135.9, 60.5)
- added R17: 100K, Resistor_THT:R_Axial_DIN0207_L6.3mm_D2.5mm_P7.62mm_Horizontal, F.Cu at (135.9, 64.5)
- added R18: 470R, Resistor_THT:R_Axial_DIN0207_L6.3mm_D2.5mm_P7.62mm_Horizontal, F.Cu at (135.9, 68.6)
- added R19: 150K, Resistor_THT:R_Axial_DIN0207_L6.3mm_D2.5mm_P7.62mm_Horizontal, F.Cu at (135.9, 72.7)
- added R2: 22K, Resistor_THT:R_Axial_DIN0207_L6.3mm_D2.5mm_P7.62mm_Horizontal, F.Cu at (190.5, 40.2)
- added R20: 10K, Resistor_THT:R_Axial_DIN0207_L6.3mm_D2.5mm_P7.62mm_Horizontal, F.Cu at (135.9, 76.7)
- added R21: 22K, Resistor_THT:R_Axial_DIN0207_L6.3mm_D2.5mm_P7.62mm_Horizontal, F.Cu at (135.9, 80.8)
- added R22: 22K, Resistor_THT:R_Axial_DIN0207_L6.3mm_D2.5mm_P7.62mm_Horizontal, F.Cu at (199.3, 82.8)
- added R23: 10K, Resistor_THT:R_Axial_DIN0207_L6.3mm_D2.5mm_P7.62mm_Horizontal, F.Cu at (199.3, 86.8)
- added R24: 47K, Resistor_THT:R_Axial_DIN0207_L6.3mm_D2.5mm_P7.62mm_Horizontal, F.Cu at (199.3, 90.8)
- added R25: 10K, Resistor_THT:R_Axial_DIN0207_L6.3mm_D2.5mm_P7.62mm_Horizontal, F.Cu at (199.3, 94.9)
- added R26: 100K, Resistor_THT:R_Axial_DIN0207_L6.3mm_D2.5mm_P7.62mm_Horizontal, F.Cu at (199.3, 99.0)
- added R27: 15K, Resistor_THT:R_Axial_DIN0207_L6.3mm_D2.5mm_P7.62mm_Horizontal, F.Cu at (199.3, 103.0)
- added R28: 10K, Resistor_THT:R_Axial_DIN0207_L6.3mm_D2.5mm_P7.62mm_Horizontal, F.Cu at (199.3, 107.0)
- added R29: 1K, Resistor_THT:R_Axial_DIN0207_L6.3mm_D2.5mm_P7.62mm_Horizontal, F.Cu at (199.3, 111.1)
- added R3: 100K, Resistor_THT:R_Axial_DIN0207_L6.3mm_D2.5mm_P7.62mm_Horizontal, F.Cu at (190.5, 44.3)
- added R30: 100K, Resistor_THT:R_Axial_DIN0207_L6.3mm_D2.5mm_P7.62mm_Horizontal, F.Cu at (199.3, 115.2)
- added R31: 100K, Resistor_THT:R_Axial_DIN0207_L6.3mm_D2.5mm_P7.62mm_Horizontal, F.Cu at (159.4, 36.2)
- added R32: 22K, Resistor_THT:R_Axial_DIN0207_L6.3mm_D2.5mm_P7.62mm_Horizontal, F.Cu at (159.4, 40.2)
- added R33: 1K5, Resistor_THT:R_Axial_DIN0207_L6.3mm_D2.5mm_P7.62mm_Horizontal, F.Cu at (159.4, 44.3)
- added R34: 100K, Resistor_THT:R_Axial_DIN0207_L6.3mm_D2.5mm_P7.62mm_Horizontal, F.Cu at (159.4, 48.4)
- added R35: 470R, Resistor_THT:R_Axial_DIN0207_L6.3mm_D2.5mm_P7.62mm_Horizontal, F.Cu at (159.4, 52.4)
- added R36: 22K, Resistor_THT:R_Axial_DIN0207_L6.3mm_D2.5mm_P7.62mm_Horizontal, F.Cu at (159.4, 56.5)
- added R37: 10K, Resistor_THT:R_Axial_DIN0207_L6.3mm_D2.5mm_P7.62mm_Horizontal, F.Cu at (159.4, 60.5)
- added R38: 0R-1K, Resistor_THT:R_Axial_DIN0207_L6.3mm_D2.5mm_P7.62mm_Horizontal, F.Cu at (159.4, 64.5)
- added R39: 470K, Resistor_THT:R_Axial_DIN0207_L6.3mm_D2.5mm_P7.62mm_Horizontal, F.Cu at (159.4, 68.6)
- added R4: 100K, Resistor_THT:R_Axial_DIN0207_L6.3mm_D2.5mm_P7.62mm_Horizontal, F.Cu at (190.5, 48.4)
- added R40: 470K, Resistor_THT:R_Axial_DIN0207_L6.3mm_D2.5mm_P7.62mm_Horizontal, F.Cu at (159.4, 72.7)
- added R41: 33K-NC, Resistor_THT:R_Axial_DIN0207_L6.3mm_D2.5mm_P7.62mm_Horizontal, F.Cu at (159.4, 76.7)
- added R5: 1K8, Resistor_THT:R_Axial_DIN0207_L6.3mm_D2.5mm_P7.62mm_Horizontal, F.Cu at (190.5, 52.4)
- added R6: 470K, Resistor_THT:R_Axial_DIN0207_L6.3mm_D2.5mm_P7.62mm_Horizontal, F.Cu at (190.5, 56.5)
- added R7: 10K, Resistor_THT:R_Axial_DIN0207_L6.3mm_D2.5mm_P7.62mm_Horizontal, F.Cu at (190.5, 60.5)
- added R8: 47K, Resistor_THT:R_Axial_DIN0207_L6.3mm_D2.5mm_P7.62mm_Horizontal, F.Cu at (190.5, 64.5)
- added R9: 47K, Resistor_THT:R_Axial_DIN0207_L6.3mm_D2.5mm_P7.62mm_Horizontal, F.Cu at (190.5, 68.6)
- added RV1: 50K-B PREAMP, DIY_jorge:Pot Alpha 16mm, B.Cu at (23.8, 84.9)
- added RV2: 50K-B VOL, DIY_jorge:Pot Alpha 16mm, B.Cu at (55.9, 84.9)
- added RV3: 50K-B WAH, DIY_jorge:Pot Alpha 16mm, B.Cu at (83.8, 84.9)
- added SW1: TONE, DIY_jorge:SW_SPDT_V2, B.Cu at (71.1, 91.4)
- added SW2: SW_DPDT - OCT, DIY_jorge:SW_DPDT, B.Cu at (38.1, 91.4)
Other:
- board outline added: 90 x 90 mm
